Commit message: migrate to jazzy

File: urdf/xacros/psen_scan.urdf.xacro (robot description, xacro)
@@ -1,5 +1,5 @@
 <?xml version="1.0"?>
 <robot xmlns:xacro="http://ros.org/wiki/xacro">
-  <xacro:macro name="psen_scan" params="prefix">
+  <xacro:macro name="psen_scan" params="prefix parent *origin">
     <xacro:property name="mass" value="1.53" /> <!-- src datasheet p 96 -->
     <xacro:property name="radius" value="0.051" /> <!-- src datasheet p 96 -->
@@ -7,4 +7,9 @@
     <xacro:property name="dist_scanning_plane_top" value="0.0377" /> <!-- src datasheet p 96 -->
     <xacro:property name="dist_scanning_axis_rear" value="0.0525" /> <!-- src datasheet p 96 -->
+    <joint name="${prefix}_joint" type="fixed">
+      <parent link="reference_link" />
+      <child link="${prefix}_mount_link" />
+      <xacro:insert_block name="origin" />
+    </joint>
     <!-- Location of mounting point at the lower back of device -->
     <link name="${prefix}_mount_link"/>
@@ -17,6 +22,7 @@
     <link name="${prefix}_body_link">
       <visual>
+        <origin xyz="-0.016 0 -0.039" rpy="0 0 3.14" />
         <geometry>
-          <cylinder radius="${radius}" length="${height}" />
+          <mesh filename="package://psen_scan_v2/urdf/meshes/PSENscan.dae" scale="0.001 0.001 0.001"/>
         </geometry>
         <material name="pilz_yellow" >
@@ -25,6 +31,7 @@
       </visual>
       <collision>
+        <origin xyz="-0.016 0 -0.039" rpy="0 0 3.14" />
         <geometry>
-          <cylinder radius="${radius}" length="${height}" />
+          <mesh filename="package://psen_scan_v2/urdf/meshes/PSENscan.dae" scale="0.001 0.001 0.001"/>
         </geometry>
       </collision>
@@ -43,6 +50,5 @@
     </joint>
     <!-- This is the location of the laser scan -->
-    <link name="${prefix}">
-    </link>
+    <link name="${prefix}"/>
   </xacro:macro>
 </robot>
